File: Schematics/Backplane/Backplane.kicad_pcb (KiCad board)
At the start: 2 copper layers, 69.5 x 119 mm, 18 parts, among them J1 Edge Connector (SLOT 1), J2 Edge Connector (SLOT 2), J3 Edge Connector (SLOT 3), J4 Edge Connector (SLOT 4), J5 Edge Connector (SLOT 5), J6 Edge Connector (SLOT 6)

Commit message: Current Updated Backplance
Did the wiring for the PCB. Not sure how to properly connect the edge connectors to the new connector (they don't want to connect)
Parts:
- removed the J1 at (32.8, 9.42)
- removed the J2 at (32.8, 29.4)
- removed the J3 at (32.8, 49.4)
- removed the J4 at (32.8, 69.4)
- removed the J5 at (32.8, 89.4)
- removed J6: Edge Connector (SLOT 6), footprints:AMPHENOL_10018784-10210TLF
- added J1: Stack Female Edge Connector, footprints:AMPHENOL_10018784-10210TLF, F.Cu at (33.4, 9.49)
- added J1: Edge Connector (SLOT 1), footprints:AMPHENOL_10018784-10210TLF, F.Cu at (239.8, 25.9)
- added J2: Stack Female Edge Connector, footprints:AMPHENOL_10018784-10210TLF, F.Cu at (33.4, 29.5)
- added J2: Edge Connector (SLOT 2), footprints:AMPHENOL_10018784-10210TLF, F.Cu at (239.8, 45.9)
- added J3: Edge Connector (SLOT 3), footprints:AMPHENOL_10018784-10210TLF, F.Cu at (239.8, 65.9)
- added J3: Stack Female Edge Connector, footprints:AMPHENOL_10018784-10210TLF, F.Cu at (33.4, 49.8)
- added J4: Edge Connector (SLOT 4), footprints:AMPHENOL_10018784-10210TLF, F.Cu at (239.8, 85.9)
- added J4: Stack Female Edge Connector, footprints:AMPHENOL_10018784-10210TLF, F.Cu at (33.4, 69.5)
- added J5: Stack Female Edge Connector, footprints:AMPHENOL_10018784-10210TLF, F.Cu at (33.4, 89.8)
- added J5: Edge Connector (SLOT 5), footprints:AMPHENOL_10018784-10210TLF, F.Cu at (239.8, 105.9)
- added R1: 120R, Resistor_SMD:R_0805_2012Metric_Pad1.20x1.40mm_HandSolder, B.Cu at (236.3, 18.9)
- added R2: 120R, Resistor_SMD:R_0805_2012Metric_Pad1.20x1.40mm_HandSolder, B.Cu at (232.6, 132.8)
- added REF**: CONN_GT8E-6P-2H(55), footprints:CONN_GT8E-8P-2H(55), F.Cu at (35.5, 112.0)
- moved R2 5.10 mm to (20.5, 116.5)
Connections:
- net CAN_H renamed CAN_+
- net CAN_L renamed CAN_-
Routing:
- net GND: track 0.00 -> 288.5 mm
- net BATT_A: track 237.6 -> 458.5 mm
- net 3.3V_A: track 189.0 -> 370.9 mm, vias 6 -> 10
- net 24V_A: track 0.00 -> 135.2 mm
- net CAN_L: track 0.00 -> 125.7 mm
- net CAN_H: track 0.00 -> 123.4 mm
- net 5.0V_A: track 199.2 -> 315.8 mm, vias 6 -> 7
- net CAN_-: track 125.7 -> 102.8 mm
- net CAN_+: track 123.4 -> 105.1 mm
- net (no net): track 0.00 -> 13.2 mm
Other:
- board size 69.5 x 119 mm -> 276.5 x 135.5 mm
