File: Schematics/Power_Module/battery_charger.kicad_sch (KiCad schematic)
At the start: 0 parts

Commit message: adding power ORing circuit
Parts:
- added U14: MAX1873SEEE+T, Package_SO:QSOP-16_3.9x4.9mm_P0.635mm, symbol Battery_Management:MAX1873SEEE
Changed lines of the file:
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@@
 	(generator_version "8.0")
 	(paper "A4")
+	(symbol
+		(lib_id "Battery_Management:MAX1873SEEE")
+		(at 134.62 91.44 0)
+		(unit 1)
+		(exclude_from_sim no)
+		(in_bom yes)
+		(on_board yes)
+		(dnp no)
+		(fields_autoplaced yes)
+		(property "Reference" "U14"
+			(at 136.8141 73.66 0)
+			(effects
+				(font
+					(size 1.27 1.27)
+				)
+				(justify left)
+			)
+		)
+		(property "Value" "MAX1873SEEE+T"
+			(at 136.8141 76.2 0)
+			(effects
+				(font
+					(size 1.27 1.27)
+				)
+				(justify left)
+			)
+		)
+		(property "Footprint" "Package_SO:QSOP-16_3.9x4.9mm_P0.635mm"
+			(at 134.62 109.22 0)
+			(effects
+				(font
+					(size 1.27 1.27)
+				)
+				(hide yes)
+			)
+		)
+		(property "Datasheet" "${KIPRJMOD}/../../Datasheets/max1873.pdf"
+			(at 139.7 91.44 0)
+			(effects
+				(font
+					(size 1.27 1.27)
+				)
+				(hide yes)
+			)
+		)
+		(property "Description" "Charger for 3 lithium-ion (Li+), 7/9 NickelCadium (NiCD) cells or 7/9 NickelMetalHydride (NiMH), 9 to 28V VDD, -40 to +85 degree Celsius, QSOP-16"
+			(at 134.62 91.44 0)
+			(effects
+				(font
+					(size 1.27 1.27)
+				)
+				(hide yes)
+			)
+		)
+		(property "LCSC" "C34333"
+			(at 134.62 91.44 0)
+			(effects
+				(font
+					(size 1.27 1.27)
+				)
+				(hide yes)
+			)
+		)
+		(pin "12"
+		)
+		(pin "2"
+		)
+		(pin "6"
+		)
+		(pin "9"
+		)
+		(pin "11"
+		)
+		(pin "5"
+		)
+		(pin "1"
+		)
+		(pin "10"
+		)
+		(pin "8"
+		)
+		(pin "7"
+		)
+		(pin "14"
+		)
+		(pin "13"
+		)
+		(pin "3"
+		)
+		(pin "15"
+		)
+		(pin "16"
+		)
+		(pin "4"
+		)
+		(instances
+			(project ""
+				(path "/11b1f19b-ce82-4fce-baf6-0357ef2e3f24/9cd93e14-529d-4d54-8401-cafe904bdef2"
+					(reference "U14")
+					(unit 1)
+				)
+			)
+		)
+	)
 )
