File: Schematics/Power_Module/Power_Module.kicad_sch (KiCad schematic)
At the start: 0 parts

Commit message: completed all power traces, finalizing signal traces
Changed lines of the file:
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@@
 		(comment 4 "GRID = 0.635mm")
 	)
-	(text_box "TODO\n - Add GSE_SENSE and 24V_CURR_SENSE\n - Review COMP C and R\n - Review 24V current sensing\n - find a few small decen size buck caps (https://www.digikey.ca/en/products/filter/aluminum-electrolytic-capacitors/w%C3%BCrth-elektronik/58?s=N4IgjCBcoCwGxVAYygMwIYBsDOBTANCAPZQDa4AzABwAMVIhYATEzRIzdQOwgC6hABwAuUEAGUhAJwCWAOwDmIAL6E4ATkQgUkDDgLEyIGDTUVTfQSMjipcxSpCsuG6FrRY8hEpHJgaAAgA1BnA4IJCKAFZwwiZo4MJIgOD%2BEGFRAFVZaSEAeVQAWVx0bABXSVxlQgBaCFdtXU8QADdZKClS-W9yLgomCzSrGxkFZSUlIA)\n - double check the voltage devider resisters can take the current\n - add a cap to 24V_GSE for energy storage\n - review LCSC, noticed one was out of stock"
+	(text_box "TODO\n - Add GSE_SENSE and 24V_CURR_SENSE\n - Review COMP C and R\n - Review 24V current sensing\n - add a cap to 24V_GSE for energy storage\n - switch to ceramic bulk caps\n - review LCSC, noticed one was out of stock"
 		(exclude_from_sim no)
 		(at 113.03 115.0112 0)
