File: Schematics/Hybrid_Backplane/Backplane.kicad_sch (KiCad schematic)
At the start: 21 parts, among them J1 Edge Connector (SLOT 1), J2 Edge Connector (SLOT 2), J3 Edge Connector (SLOT 3), J4 Edge Connector (SLOT 4), J5 Edge Connector (SLOT 5), J6 Conn_01x06

Commit message: add nano connector for xpand, adjust routing
Parts:
- J6: footprint footprints:CONN_SD-43045-001_06_MOL -> footprints:CONN_SD-105314-100_06_MOL
Changed lines of the file:
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@@
 			)
 		)
-		(property "Footprint" "footprints:CONN_SD-43045-001_06_MOL"
+		(property "Footprint" "footprints:CONN_SD-105314-100_06_MOL"
 			(at 139.7 74.93 0)
 			(effects
